Commit message: Update my_robot.xacro

File: Project2/my_robot/urdf/my_robot.xacro (robot description, xacro)
@@ -23,5 +23,5 @@
       <origin xyz="0 0 0" rpy=" 0 0 0"/>
       <geometry>
-        <box size=".5 .2 .2"/>
+        <box size=".4 .2 .1"/>
       </geometry>
     </collision>
@@ -29,5 +29,5 @@
       <origin xyz="0 0 0" rpy=" 0 0 0"/>
       <geometry>
-        <box size=".5 .2 .2"/>
+        <box size=".4 .2 .1"/>
       </geometry>
     </visual>
